File: hardware/gnss-7-seg-clock.kicad_pcb (KiCad board)
At the start: 2 copper layers, 225 x 63.5 mm, 90 parts, among them J1 USB4105-GF-A, J2 Conn_Coaxial, J3 Conn_01x03, SW1 SW_Push, SW2 SW_Push, SW3 SW_Push, SW4 SW_Push, SW5 SW_Push, U1 SA15-11GWA, U10 RP2040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

Commit message: Reduce output current of TLC5925 (22 mA -> 9.9 mA)
It was too high for LSD150BAG-101.
Parts:
- R1, R2, R3: value 1k -> 2.2k
Changed lines of the file:
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@@
 			)
 		)
-		(property "Value" "1k"
+		(property "Value" "2.2k"
 			(at 0 1.17 0)
 			(layer "F.Fab")
@@
 			)
 		)
-		(property "Value" "1k"
+		(property "Value" "2.2k"
 			(at 0 1.17 0)
 			(layer "F.Fab")
@@
 			)
 		)
-		(property "Value" "1k"
+		(property "Value" "2.2k"
 			(at 0 1.17 0)
 			(layer "F.Fab")

Commit message: Hardware Rev.A2 (for reflow soldering)
Parts:
- C1, C10, C11, C14, C15, C16, C17, C18, C19, C2, C20, C21, C3, C4, C5, C6, C7, C8, C9: footprint Capacitor_SMD:C_0402_1005Metric_Pad0.74x0.62mm_HandSolder -> Capacitor_SMD:C_0402_1005Metric
- C12, C13: footprint Capacitor_SMD:C_0805_2012Metric_Pad1.18x1.45mm_HandSolder -> Capacitor_SMD:C_0805_2012Metric
- D1: footprint Diode_SMD:D_0402_1005Metric_Pad0.77x0.64mm_HandSolder -> Diode_SMD:D_0402_1005Metric
- D2, D3, D4, D5, D6, D7: footprint LED_SMD:LED_0402_1005Metric_Pad0.77x0.64mm_HandSolder -> LED_SMD:LED_0402_1005Metric
- J1: footprint gnss-7-seg-clock:USB_C_Receptacle_GCT_USB4105-xx-A_16P_TopMnt_Horizontal_HandSolder -> gnss-7-seg-clock:USB_C_Receptacle_GCT_USB4105-xx-A_16P_TopMnt_Horizontal
- L1: footprint Inductor_SMD:L_0402_1005Metric_Pad0.77x0.64mm_HandSolder -> Inductor_SMD:L_0402_1005Metric
- R1, R10, R11, R12, R13, R14, R15, R16, R17, R18, R19, R2, R20, R21, R22, R3, R4, R5, R6, R7, R8, R9: footprint Resistor_SMD:R_0402_1005Metric_Pad0.72x0.64mm_HandSolder -> Resistor_SMD:R_0402_1005Metric
- SW1, SW2, SW3, SW4, SW5: footprint gnss-7-seg-clock:SW_SPST_PTS810_HandSolder -> Button_Switch_SMD:SW_SPST_PTS810
- U10: footprint gnss-7-seg-clock:QFN-56-1EP_7x7mm_P0.4mm_EP3.2x3.2mm_HandSolder -> Package_DFN_QFN:QFN-56-1EP_7x7mm_P0.4mm_EP3.2x3.2mm_ThermalVias
- U11: footprint Package_TO_SOT_SMD:TSOT-23-5_HandSoldering -> Package_TO_SOT_SMD:TSOT-23-5
- Y1: footprint Crystal:Crystal_SMD_3225-4Pin_3.2x2.5mm_HandSoldering -> Crystal:Crystal_SMD_3225-4Pin_3.2x2.5mm
Other:
- board text removed: "For JLCPCB 2D barcode"
