File: hardware/gnss-7-seg-clock.kicad_sch (KiCad schematic)
At the start: 90 parts, among them J1 USB4105-GF-A, J2 Conn_Coaxial, J3 Conn_01x03, SW1 SW_Push, SW2 SW_Push, SW3 SW_Push, SW4 SW_Push, SW5 SW_Push, U1 SA15-11GWA, U10 RP2040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

Commit message: Reduce output current of TLC5925 (22 mA -> 9.9 mA)
It was too high for LSD150BAG-101.
Parts:
- R1, R2, R3: value 1k -> 2.2k
Other:
- note added: "Setting the output current of TLC5925 Iout = (1.21 / Rext) * 18 Iout = 9.9 mA (Rext = 2.2k) https://www.ti.com/lit/gpn/tlc5925"
Changed lines of the file:
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@@
 	(title_block
 		(title "GNSS Seven-segment Clock")
-		(date "2025-01-25")
-		(rev "A")
+		(date "2025-01-31")
+		(rev "A2")
 	)
 	(junction
@@
 		)
 	)
+	(text "Setting the output current of TLC5925\nIout = (1.21 / Rext) * 18\nIout = 9.9 mA (Rext = 2.2k)\nhttps://www.ti.com/lit/gpn/tlc5925"
+		(exclude_from_sim no)
+		(at 12.954 89.154 0)
+		(effects
+			(font
+				(size 1.27 1.27)
+			)
+			(justify left)
+		)
+	)
 	(label "GNSS_EXTINT"
 		(at 215.9 214.63 180)
@@
 			)
 		)
-		(property "Value" "1k"
+		(property "Value" "2.2k"
 			(at 34.29 71.1199 0)
 			(effects
@@
 			)
 		)
-		(property "Value" "1k"
+		(property "Value" "2.2k"
 			(at 237.49 71.1199 0)
 			(effects
@@
 			)
 		)
-		(property "Value" "1k"
+		(property "Value" "2.2k"
 			(at 135.89 71.1199 0)
 			(effects

Commit message: Re-save project with KiCad 9.0.0
Changed lines of the file:
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@@
 (kicad_sch
-	(version 20231120)
+	(version 20250114)
 	(generator "eeschema")
-	(generator_version "8.0")
+	(generator_version "9.0")
 	(paper "A3")
 	(title_block
@@
 		(rev "A2")
 	)
+	(text "Setting the output current of TLC5925\nIout = (1.21 / Rext) * 18\nIout = 9.9 mA (Rext = 2.2k)\nhttps://www.ti.com/lit/gpn/tlc5925"
+		(exclude_from_sim no)
+		(at 12.954 89.154 0)
+		(effects
+			(font
+				(size 1.27 1.27)
+			)
+			(justify left)
+		)
+	)
 	(junction
 		(at 312.42 114.3)
@@
 		)
 	)
-	(text "Setting the output current of TLC5925\nIout = (1.21 / Rext) * 18\nIout = 9.9 mA (Rext = 2.2k)\nhttps://www.ti.com/lit/gpn/tlc5925"
-		(exclude_from_sim no)
-		(at 12.954 89.154 0)
-		(effects
-			(font
-				(size 1.27 1.27)
-			)
-			(justify left)
-		)
-	)
 	(label "GNSS_EXTINT"
 		(at 215.9 214.63 180)
@@
 		)
 	)
+	(embedded_fonts no)
 )

Commit message: Update W25Q32JVSS footprint
see also: https://gitlab.com/kicad/libraries/kicad-footprint-generator/-/merge_requests/1384
Parts:
- U12: footprint Package_SO:SOIC-8_5.275x5.275mm_P1.27mm -> Package_SO:SOIC-8_5.3x5.3mm_P1.27mm; symbol Memory_Flash:W25Q16JVSS -> Memory_Flash:W25Q32JVSS
Other:
- moved on the sheet: U12
Changed lines of the file:
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@@
 	)
 	(symbol
-		(lib_id "Memory_Flash:W25Q16JVSS")
+		(lib_id "Memory_Flash:W25Q32JVSS")
 		(at 76.2 251.46 0)
 		(unit 1)
@@
 		(fields_autoplaced yes)
 		(property "Reference" "U12"
-			(at 85.09 250.1899 0)
+			(at 87.63 250.1899 0)
 			(effects
 				(font
@@
 		)
 		(property "Value" "W25Q32JVSS"
-			(at 85.09 252.7299 0)
+			(at 87.63 252.7299 0)
 			(effects
 				(font
@@
 			)
 		)
-		(property "Footprint" "Package_SO:SOIC-8_5.275x5.275mm_P1.27mm"
+		(property "Footprint" "Package_SO:SOIC-8_5.3x5.3mm_P1.27mm"
 			(at 76.2 251.46 0)
 			(effects
@@
 			)
 		)
-		(property "Datasheet" ""
+		(property "Datasheet" "http://www.winbond.com/resource-files/w25q32jv%20revg%2003272018%20plus.pdf"
 			(at 76.2 251.46 0)
 			(effects
@@
 			)
 		)
-		(property "Description" "4Mb Serial Flash Memory, Standard/Dual/Quad SPI, SOIC-8"
+		(property "Description" "32Mbit / 4MiB Serial Flash Memory, Standard/Dual/Quad SPI, 2.7-3.6V, SOIC-8 (208 mil)"
 			(at 76.2 251.46 0)
 			(effects
